File: kicad/mainboard/audioplayer.sch (KiCad schematic (older format))
At the start: 33 parts, among them J1 Panel, J2 Charge_USB, J3 SPK, J4 RFID, SW1 POWER, U1 PB-500, U2 ESP32-nodeMCU, U3 OLED, U4 GY-521, U5 VS1053/SD_breakout, U6 ULN2003, U7 HW-323

Commit message: board rev04
Parts:
- removed D1: 1N4007, Diode_THT:D_DO-41_SOD81_P10.16mm_Horizontal, symbol Diode:1N4007
- removed J2: Charge_USB, Connector_PinHeader_2.54mm:PinHeader_1x02_P2.54mm_Vertical, symbol Connector_Generic:Conn_01x02
- removed SW1: POWER, Connector_PinHeader_2.54mm:PinHeader_1x02_P2.54mm_Vertical, symbol Switch:SW_SPST
- added J2: Conn_02x04_Odd_Even, Connector_PinHeader_2.54mm:PinHeader_2x04_P2.54mm_Vertical, symbol Connector_Generic:Conn_02x04_Odd_Even
- added R4, R5: ?, Resistor_THT:R_Axial_DIN0204_L3.6mm_D1.6mm_P7.62mm_Horizontal, symbol Device:R
- added R?: 47k, Resistor_THT:R_Axial_DIN0204_L3.6mm_D1.6mm_P7.62mm_Horizontal, symbol Device:R
- added TP4: R, Connector_PinHeader_2.54mm:PinHeader_1x01_P2.54mm_Vertical, symbol Connector:TestPoint
Connections:
- net labels added: USB+
- net labels removed: SW4
- wire segments 200 -> 227
Other:
- note added: "1: USB+\n2: USB- (GND)\n3: PWR SW\n4: PWR SW (VBAT)\n5: Full LED (+)\n6: Full LED (-)\n7: Charge LED (+)\n8: Charge LED (-)"
- note added: "headphone switch"
- note removed: "Power supply\nfrom USB jack"
Changed lines of the file:
@@
 Text Label 6700 800  2    50   ~ 0
 AMP_ENABLE
-$Comp
-L Switch:SW_SPST SW1
-U 1 1 5BEEA3BD
-P 2450 4750
-F 0 "SW1" H 2450 4650 50  0000 C CNN
-F 1 "POWER" H 2450 4550 50  0000 C CNN
-F 2 "Connector_PinHeader_2.54mm:PinHeader_1x02_P2.54mm_Vertical" H 2450 4750 50  0001 C CNN
-F 3 "" H 2450 4750 50  0001 C CNN
-	1    2450 4750
-	1    0    0    -1
-$EndComp
-Wire Wire Line
-	2200 4750 2250 4750
-Wire Wire Line
-	2650 4750 2800 4750
-Wire Wire Line
-	2800 4750 2800 4850
-$Comp
-L power:GND #PWR06
-U 1 1 5BEF6B43
-P 2800 4850
-F 0 "#PWR06" H 2800 4600 50  0001 C CNN
-F 1 "GND" H 2800 4700 50  0000 C CNN
-F 2 "" H 2800 4850 50  0000 C CNN
-F 3 "" H 2800 4850 50  0000 C CNN
-	1    2800 4850
-	1    0    0    -1
-$EndComp
 Text GLabel 5700 3250 2    50   Input ~ 0
 LED1
@@
 Text GLabel 4000 2600 0    50   Input ~ 0
 LED3
-Text GLabel 3300 3250 0    50   Input ~ 0
+Text GLabel 3450 3250 0    50   Input ~ 0
 SW1
-Text GLabel 3000 3350 0    50   Input ~ 0
+Text GLabel 3450 3350 0    50   Input ~ 0
 SW2
-Text GLabel 3300 3050 0    50   Input ~ 0
+Text GLabel 3450 3050 0    50   Input ~ 0
 SW3
 Wire Wire Line
@@
 Text Label 2300 3300 1    50   ~ 0
 LOW_BATT
-$Comp
-L Connector_Generic:Conn_01x02 J2
-U 1 1 5BE39FB9
-P 3900 4500
-F 0 "J2" H 3979 4492 50  0000 L CNN
-F 1 "Charge_USB" H 3979 4401 50  0000 L CNN
-F 2 "Connector_PinHeader_2.54mm:PinHeader_1x02_P2.54mm_Vertical" H 3900 4500 50  0001 C CNN
-F 3 "~" H 3900 4500 50  0001 C CNN
-	1    3900 4500
-	1    0    0    -1
-$EndComp
-Text Notes 3600 4850 0    50   ~ 0
-Power supply\nfrom USB jack
+Text Notes 3800 4750 0    50   ~ 0
+1: USB+\n2: USB- (GND)\n3: PWR SW\n4: PWR SW (VBAT)\n5: Full LED (+)\n6: Full LED (-)\n7: Charge LED (+)\n8: Charge LED (-)
 $Comp
 L Connector:Conn_01x04_Male J3
@@
 	1300 2950 1300 2850
 Wire Wire Line
-	1300 3250 1300 4400
+	1300 3250 1300 3700
 Text Notes 950  2850 0    50   ~ 0
 4.3V battery -> 1.0V ADC
@@
 Wire Wire Line
 	5450 3250 5700 3250
-Text Label 3500 6350 0    50   ~ 0
+Text Label 3500 6650 0    50   ~ 0
 LED1_OD
+Text Label 3500 6550 0    50   ~ 0
+LED2_OD
 Text Label 3500 6450 0    50   ~ 0
-LED2_OD
-Text Label 3500 6550 0    50   ~ 0
 LED3_OD
 Wire Wire Line
-	3450 6550 3900 6550
+	3450 6550 4100 6550
 Wire Wire Line
 	3450 6350 4200 6350
@@
 Text GLabel 2600 6350 0    50   Input ~ 0
 LED4
-Text GLabel 3000 3150 0    50   Input ~ 0
-SW4
 Wire Wire Line
 	1950 2850 4350 2850
-Text GLabel 4900 6850 2    50   Input ~ 0
-SW4
-Text Label 3500 6650 0    50   ~ 0
+Text Label 3500 6350 0    50   ~ 0
 LED4_OD
 Wire Wire Line
@@
 	3450 6450 4150 6450
 Wire Wire Line
-	3900 6550 3900 6750
-Wire Wire Line
-	3900 6750 4350 6750
-Wire Wire Line
-	3450 6650 3850 6650
-Wire Wire Line
-	3850 6650 3850 6850
-Wire Wire Line
-	3850 6850 4350 6850
+	4100 6550 4100 6750
+Wire Wire Line
+	4100 6750 4350 6750
+Wire Wire Line
+	3450 6650 4050 6650
+Wire Wire Line
+	4050 6650 4050 6850
+Wire Wire Line
+	4050 6850 4350 6850
 Wire Wire Line
 	2600 6950 2600 6850
@@
 Wire Wire Line
 	3550 6150 3550 6100
-$Comp
-L Diode:1N4007 D1
-U 1 1 5C1A04B7
-P 3200 4500
-F 0 "D1" H 3200 4716 50  0000 C CNN
-F 1 "1N4007" H 3200 4625 50  0000 C CNN
-F 2 "Diode_THT:D_DO-41_SOD81_P10.16mm_Horizontal" H 3200 4325 50  0001 C CNN
-F 3 "http://www.vishay.com/docs/88503/1n4001.pdf" H 3200 4500 50  0001 C CNN
-	1    3200 4500
-	1    0    0    -1
-$EndComp
-Wire Wire Line
-	2200 4500 3050 4500
-Wire Wire Line
-	3350 4500 3700 4500
+Wire Wire Line
+	2200 4500 3000 4500
 $Comp
 L Device:R R6
@@
 $EndComp
 Wire Wire Line
-	3000 3150 3500 3150
-Wire Wire Line
-	3300 3050 3600 3050
-Wire Wire Line
-	3000 3350 3700 3350
-Wire Wire Line
-	3300 3250 3800 3250
+	3450 3050 3600 3050
+Wire Wire Line
+	3450 3350 3700 3350
+Wire Wire Line
+	3450 3250 3800 3250
 Wire Wire Line
 	3800 3500 3800 3250
@@
 Wire Wire Line
 	3500 3500 3500 3150
-Connection ~ 3500 3150
 Wire Wire Line
 	3500 3150 4350 3150
@@
 Wire Wire Line
 	4200 6950 4350 6950
-Wire Wire Line
-	4850 6850 4900 6850
 Wire Wire Line
 	4900 7000 4900 6950
@@
 L power:GND #PWR0121
 U 1 1 5C1A1D3C
-P 3450 4700
-F 0 "#PWR0121" H 3450 4450 50  0001 C CNN
-F 1 "GND" H 3450 4550 50  0000 C CNN
-F 2 "" H 3450 4700 50  0000 C CNN
-F 3 "" H 3450 4700 50  0000 C CNN
-	1    3450 4700
-	1    0    0    -1
-$EndComp
-Wire Wire Line
-	3450 4700 3450 4600
-Wire Wire Line
-	3450 4600 3700 4600
+P 3950 5100
+F 0 "#PWR0121" H 3950 4850 50  0001 C CNN
+F 1 "GND" H 3950 4950 50  0000 C CNN
+F 2 "" H 3950 5100 50  0000 C CNN
+F 3 "" H 3950 5100 50  0000 C CNN
+	1    3950 5100
+	0    -1   -1   0
+$EndComp
 Wire Wire Line
 	1700 5150 1700 5200
@@
 Wire Wire Line
 	2300 2700 2650 2700
+Wire Wire Line
+	4850 6850 4900 6850
+Wire Wire Line
+	4900 6850 4900 6950
+Connection ~ 4900 6950
+Wire Wire Line
+	3500 3150 2550 3150
+Wire Wire Line
+	2550 3150 2550 3300
+Connection ~ 3500 3150
+$Comp
+L power:GNDA #PWR0123
+U 1 1 5C51AD39
+P 2550 3300
+F 0 "#PWR0123" H 2550 3050 50  0001 C CNN
+F 1 "GNDA" H 2555 3127 50  0000 C CNN
+F 2 "" H 2550 3300 50  0001 C CNN
+F 3 "" H 2550 3300 50  0001 C CNN
+	1    2550 3300
+	1    0    0    -1
+$EndComp
+Text Notes 2550 3150 0    50   ~ 0
+headphone switch
+$Comp
+L Device:R R4
+U 1 1 5C6A100C
+P 2600 5550
+F 0 "R4" H 2700 5600 50  0000 C CNN
+F 1 "?" H 2750 5500 50  0000 C CNN
+F 2 "Resistor_THT:R_Axial_DIN0204_L3.6mm_D1.6mm_P7.62mm_Horizontal" V 2530 5550 50  0001 C CNN
+F 3 "~" H 2600 5550 50  0001 C CNN
+	1    2600 5550
+	0    1    1    0
+$EndComp
+$Comp
+L Device:R R5
+U 1 1 5C6B7954
+P 2600 5350
+F 0 "R5" H 2700 5400 50  0000 C CNN
+F 1 "?" H 2750 5300 50  0000 C CNN
+F 2 "Resistor_THT:R_Axial_DIN0204_L3.6mm_D1.6mm_P7.62mm_Horizontal" V 2530 5350 50  0001 C CNN
+F 3 "~" H 2600 5350 50  0001 C CNN
+	1    2600 5350
+	0    1    1    0
+$EndComp
+Wire Wire Line
+	2450 5550 2250 5550
+Wire Wire Line
+	2250 5350 2450 5350
+$Comp
+L Connector_Generic:Conn_02x04_Odd_Even J2
+U 1 1 5C6E7F83
+P 3450 5200
+F 0 "J2" H 3500 5517 50  0000 C CNN
+F 1 "Conn_02x04_Odd_Even" H 3500 5426 50  0000 C CNN
+F 2 "Connector_PinHeader_2.54mm:PinHeader_2x04_P2.54mm_Vertical" H 3450 5200 50  0001 C CNN
+F 3 "~" H 3450 5200 50  0001 C CNN
+	1    3450 5200
+	1    0    0    -1
+$EndComp
+Wire Wire Line
+	3750 5100 3850 5100
+Wire Wire Line
+	3250 5100 3200 5100
+Wire Wire Line
+	3000 5100 3000 4500
+Wire Wire Line
+	2900 4750 2900 5200
+Wire Wire Line
+	2900 5200 3250 5200
+Wire Wire Line
+	2200 4750 2450 4750
+Connection ~ 3850 5100
+Wire Wire Line
+	3850 5100 3950 5100
+Wire Wire Line
+	2250 5350 2250 5450
+Wire Wire Line
+	3750 5300 3850 5300
+Wire Wire Line
+	3850 5550 3850 5400
+Wire Wire Line
+	3850 5400 3750 5400
+Wire Wire Line
+	2750 5550 3850 5550
+$Comp
+L Connector:TestPoint TP4
+U 1 1 5C88FD5A
+P 2200 5450
+F 0 "TP4" V 2395 5524 50  0000 C CNN
+F 1 "R" V 2304 5524 50  0000 C CNN
+F 2 "Connector_PinHeader_2.54mm:PinHeader_1x01_P2.54mm_Vertical" H 2400 5450 50  0001 C CNN
+F 3 "~" H 2400 5450 50  0001 C CNN
+	1    2200 5450
+	0    -1   -1   0
+$EndComp
+Wire Wire Line
+	2200 5450 2250 5450
+Connection ~ 2250 5450
+Wire Wire Line
+	2250 5450 2250 5550
+Wire Wire Line
+	3250 5400 3200 5400
+Wire Wire Line
+	3200 5400 3200 5100
+Connection ~ 3200 5100
+Wire Wire Line
+	3200 5100 3000 5100
+Text Label 2700 4500 0    50   ~ 0
+USB+
+$Comp
+L Device:R R?
+U 1 1 5C8AB77F
+P 2450 4950
+F 0 "R?" H 2550 5000 50  0000 C CNN
+F 1 "47k" H 2600 4900 50  0000 C CNN
+F 2 "Resistor_THT:R_Axial_DIN0204_L3.6mm_D1.6mm_P7.62mm_Horizontal" V 2380 4950 50  0001 C CNN
+F 3 "~" H 2450 4950 50  0001 C CNN
+	1    2450 4950
+	-1   0    0    1
+$EndComp
+Wire Wire Line
+	2450 4800 2450 4750
+Connection ~ 2450 4750
+Wire Wire Line
+	2450 4750 2900 4750
+$Comp
+L power:GND #PWR?
+U 1 1 5C8B9589
+P 2450 5100
+F 0 "#PWR?" H 2450 4850 50  0001 C CNN
+F 1 "GND" H 2450 4950 50  0000 C CNN
+F 2 "" H 2450 5100 50  0000 C CNN
+F 3 "" H 2450 5100 50  0000 C CNN
+	1    2450 5100
+	1    0    0    -1
+$EndComp
+Wire Wire Line
+	3250 5300 3150 5300
+Wire Wire Line
+	3150 5300 3150 5350
+Wire Wire Line
+	3150 5350 2750 5350
+Wire Wire Line
+	3850 5100 3850 5300
+Wire Wire Line
+	3750 5200 3800 5200
+Wire Wire Line
+	3800 5200 3800 4750
+Wire Wire Line
+	3800 4750 3100 4750
+Wire Wire Line
+	3100 4750 3100 3700
+Wire Wire Line
+	3100 3700 1300 3700
 Wire Bus Line
 	7050 2900 7050 4500
@@
 Wire Bus Line
 	6400 1750 6400 3550
+Connection ~ 1300 3700
+Wire Wire Line
+	1300 3700 1300 4400
 $EndSCHEMATC

Commit message: board rev04
Parts:
- gave numbers to parts that had none: 1
Changed lines of the file:
@@
 USB+
 $Comp
-L Device:R R?
+L Device:R R7
 U 1 1 5C8AB77F
 P 2450 4950
-F 0 "R?" H 2550 5000 50  0000 C CNN
+F 0 "R7" H 2550 5000 50  0000 C CNN
 F 1 "47k" H 2600 4900 50  0000 C CNN
 F 2 "Resistor_THT:R_Axial_DIN0204_L3.6mm_D1.6mm_P7.62mm_Horizontal" V 2380 4950 50  0001 C CNN
@@
 	2450 4750 2900 4750
 $Comp
-L power:GND #PWR?
+L power:GND #PWR0124
 U 1 1 5C8B9589
 P 2450 5100
-F 0 "#PWR?" H 2450 4850 50  0001 C CNN
+F 0 "#PWR0124" H 2450 4850 50  0001 C CNN
 F 1 "GND" H 2450 4950 50  0000 C CNN
 F 2 "" H 2450 5100 50  0000 C CNN

Commit message: case changed et al
Parts:
- R4: value ? -> 470
- R5: value ? -> 1k
Changed lines of the file:
@@
 P 2600 5550
 F 0 "R4" H 2700 5600 50  0000 C CNN
-F 1 "?" H 2750 5500 50  0000 C CNN
+F 1 "470" V 2600 5550 50  0000 C CNN
 F 2 "Resistor_THT:R_Axial_DIN0204_L3.6mm_D1.6mm_P7.62mm_Horizontal" V 2530 5550 50  0001 C CNN
 F 3 "~" H 2600 5550 50  0001 C CNN
@@
 P 2600 5350
 F 0 "R5" H 2700 5400 50  0000 C CNN
-F 1 "?" H 2750 5300 50  0000 C CNN
+F 1 "1k" V 2600 5350 50  0000 C CNN
 F 2 "Resistor_THT:R_Axial_DIN0204_L3.6mm_D1.6mm_P7.62mm_Horizontal" V 2530 5350 50  0001 C CNN
 F 3 "~" H 2600 5350 50  0001 C CNN
@@
 Wire Wire Line
 	3100 3700 1300 3700
+Connection ~ 1300 3700
+Wire Wire Line
+	1300 3700 1300 4400
 Wire Bus Line
 	7050 2900 7050 4500
@@
 Wire Bus Line
 	6400 1750 6400 3550
-Connection ~ 1300 3700
-Wire Wire Line
-	1300 3700 1300 4400
 $EndSCHEMATC

Commit message: WIP new board
Parts:
- removed D2: 1N4007, Diode_THT:D_DO-41_SOD81_P10.16mm_Horizontal, symbol Diode:1N4007
- removed J1: Panel, Connector_PinHeader_2.54mm:PinHeader_2x05_P2.54mm_Vertical, symbol Connector_Generic:Conn_02x05_Odd_Even
- removed J2: Conn_02x04_Odd_Even, Connector_PinHeader_2.54mm:PinHeader_2x04_P2.54mm_Vertical, symbol Connector_Generic:Conn_02x04_Odd_Even
- removed J4: RFID, Connector_PinHeader_2.54mm:PinHeader_2x05_P2.54mm_Vertical, symbol Connector_Generic:Conn_02x05_Odd_Even
- removed TP1, TP4: R, Connector_PinHeader_2.54mm:PinHeader_1x01_P2.54mm_Vertical, symbol Connector:TestPoint
- removed TP2: L, Connector_PinHeader_2.54mm:PinHeader_1x01_P2.54mm_Vertical, symbol Connector:TestPoint
- removed TP3: GNDA, Connector_PinHeader_2.54mm:PinHeader_1x01_P2.54mm_Vertical, symbol Connector:TestPoint
- removed U1: PB-500, audioplayer:adafruit-pb500-charge, symbol audioplayer:PB-500
- removed U2: ESP32-nodeMCU, audioplayer:esp32-nodemcu-noholes, symbol RF_Module:ESP32-nodeMCU
- removed U3: OLED, Connector_PinHeader_2.54mm:PinHeader_1x04_P2.54mm_Vertical, symbol audioplayer:OLED
- removed U4: GY-521, audioplayer:gy-521-noholes, symbol audioplayer:GY-521
- removed U5: VS1053/SD_breakout, audioplayer:vs1053_breakout_upside_down, symbol audioplayer:VS1053_SD_breakout
- removed U6: ULN2003, Package_SO:SOIC-16W_5.3x10.2mm_P1.27mm, symbol Transistor_Array:ULN2003
- removed U7: HW-323, audioplayer:hw-323, symbol audioplayer:HW-323
- added C1, C13, C15, C17, C18, C20, C21, C22, C23: 100n, Capacitor_THT:C_Disc_D5.1mm_W3.2mm_P5.00mm, symbol Device:C
- added C11, C16, C4: 22u, Capacitor_THT:C_Disc_D5.1mm_W3.2mm_P5.00mm, symbol Device:C
- added C12, C14, C?: 10u, symbol Device:C
- added C19: 1u, Capacitor_THT:C_Disc_D5.1mm_W3.2mm_P5.00mm, symbol Device:C
- added C24, C25: 33p, Capacitor_THT:C_Rect_L7.0mm_W2.5mm_P5.00mm, symbol Device:C
- added C26: 1u, Capacitor_THT:C_Rect_L7.0mm_W2.5mm_P5.00mm, symbol Device:C
- added C27: 47n, Capacitor_THT:C_Rect_L7.0mm_W2.5mm_P5.00mm, symbol Device:C
- added C28, C29: 10n, Capacitor_THT:C_Rect_L7.0mm_W2.5mm_P5.00mm, symbol Device:C
- added C30, C31: 4.7n, Capacitor_THT:C_Rect_L7.0mm_W2.5mm_P5.00mm, symbol Device:C
- added D1: D_Schottky, symbol Device:D_Schottky
- added D? (x2): LED, symbol Device:LED
- added F?: Fuse, symbol Device:Fuse
- added J1: USB_B, symbol Connector:USB_B
- added J2: Micro_SD_Card, symbol Connector:Micro_SD_Card
- added J?: LiPo, symbol Connector:Conn_01x02_Male
- added L1: 10u, symbol Device:L
- added L2: 1.5u, symbol Device:L
- added Q?: IRLML2244, Package_TO_SOT_SMD:SOT-23, symbol Transistor_FET:IRLML5203
- added R11: 20, Resistor_THT:R_Axial_DIN0204_L3.6mm_D1.6mm_P7.62mm_Horizontal, symbol Device:R
- added R12, R?: 1k, Resistor_THT:R_Axial_DIN0204_L3.6mm_D1.6mm_P7.62mm_Horizontal, symbol Device:R
- added R?: 470, Resistor_THT:R_Axial_DIN0204_L3.6mm_D1.6mm_P7.62mm_Horizontal, symbol Device:R
- added R?: 100k, Resistor_THT:R_Axial_DIN0204_L3.6mm_D1.6mm_P7.62mm_Horizontal, symbol Device:R
- added R?: 1M, Resistor_THT:R_Axial_DIN0204_L3.6mm_D1.6mm_P7.62mm_Horizontal, symbol Device:R
- added TP?: TestPoint_1V8, symbol Connector:TestPoint_Probe
- added TP?: TestPoint_5V5, symbol Connector:TestPoint_Probe
- added TP?: TestPoint_3V3, symbol Connector:TestPoint_Probe
- added TP?: TestPoint_Batt_Switched, symbol Connector:TestPoint_Probe
- added TP?: TestPoint_Batt, symbol Connector:TestPoint_Probe
- added TP?: TestPoint_GND, symbol Connector:TestPoint_Probe
- added U1: AMS1117-1.8, Package_TO_SOT_SMD:SOT-223-3_TabPin2, symbol Regulator_Linear:AMS1117-1.8
- added U2: MT3608, Package_TO_SOT_SMD:SOT-23-6, symbol Regulator_Switching:MT3608
- added U3: TPS63031DSK, Package_SON:WSON-10-1EP_2.5x2.5mm_P0.5mm_EP1.2x2mm, symbol Regulator_Switching:TPS63031DSK
- added U4: CP2102N-GQFN20, Package_DFN_QFN:QFN-20-1EP_3.5x3.5mm_P0.5mm_EP2x2mm, symbol audioplayer:CP2102N-GQFN20
- added U5: ESP-WROOM32, symbol audioplayer:ESP-WROOM32
- added U6: VS1053b, symbol audioplayer:VS1053b
- added U7: PAM8408, symbol audioplayer:PAM8408
- added U?: MCP73831-2-OT, Package_TO_SOT_SMD:SOT-23-5, symbol Battery_Management:MCP73831-2-OT
- added Y1: 12.288MHz, symbol Device:Crystal
- C10, C9: value 4.7n -> 100n; footprint Capacitor_THT:C_Rect_L7.0mm_W2.5mm_P5.00mm -> Capacitor_THT:C_Disc_D5.1mm_W3.2mm_P5.00mm
- C2: value 100u -> 220u; footprint Capacitor_THT:CP_Radial_D10.0mm_P5.00mm -> (none)
- C3: value C -> 10u; footprint Capacitor_THT:C_Disc_D5.1mm_W3.2mm_P5.00mm -> (none)
- C5, C7: value C -> 100n
- C6: value 100n -> 1u
- R10: value 1k -> 20
- R3: value 10k -> 47k
- R4: value 470 -> 5.6k
- R5: value 1k -> 2k
- R6: value 10 -> 100k
- R7: value 47k -> 10
Connections:
- net labels added: +1V8, +3V3, +6V, BATT, RFID_CS, RFID_RST, SW4, VOL+, VOL-
- net labels removed: +5V, +5VA, GNDA, I²C, LED1_OD, LED2_OD, LED3_OD, LED4_OD, LOW_BATT, RST, SCL, SDA, SS, USB+, VCC_AMP
- wire segments 227 -> 391
Other:
- note added: "1.8V Supply (Linear)"
- note added: "3.3V Supply (Step Up/Down)"
- note added: "6V Supply (Step Up)"
- note added: "Battery Charging"
- note added: "X7R"
- note removed: "1: USB+\n2: USB- (GND)\n3: PWR SW\n4: PWR SW (VBAT)\n5: Full LED (+)\n6: Full LED (-)\n7: Charge LED (+)\n8: Charge LED (-)"
- note removed: "Decoupling of amplifier supply"
- note removed: "LED1: playing\nLED2: \nLED3: \n\nSW1: play/pause\nSW2: Volume -\nSW3: Volume +"
- note removed: "headphone switch"
- moved on the sheet: C2, C6, C8, J3, R1, R2, R8, R9, RN1

Commit message: programming circuit
Parts:
- removed C14: 10u, symbol Device:C
- removed U4: CP2102N-GQFN20, Package_DFN_QFN:QFN-20-1EP_3.5x3.5mm_P0.5mm_EP2x2mm, symbol audioplayer:CP2102N-GQFN20
- added C?: 100n, Capacitor_THT:C_Disc_D5.1mm_W3.2mm_P5.00mm, symbol Device:C
- added Q? (x2): BC546, Package_TO_SOT_THT:TO-92_Inline, symbol Transistor_BJT:BC546
- added R? (x3): 10k, Resistor_THT:R_Axial_DIN0204_L3.6mm_D1.6mm_P7.62mm_Horizontal, symbol Device:R
- added U?: CP2102N-A01-GQFN24, Package_DFN_QFN:QFN-24-1EP_4x4mm_P0.5mm_EP2.6x2.6mm, symbol Interface_USB:CP2102N-A01-GQFN24
- C11, C16, C19, C4, C6: footprint Capacitor_THT:C_Disc_D5.1mm_W3.2mm_P5.00mm -> Capacitor_SMD:C_1206_3216Metric_Pad1.42x1.75mm_HandSolder
- C12: value 10u -> 22u; footprint (none) -> Capacitor_SMD:C_1206_3216Metric_Pad1.42x1.75mm_HandSolder
- C3: footprint (none) -> Capacitor_SMD:C_1206_3216Metric_Pad1.42x1.75mm_HandSolder
- C8: footprint Capacitor_THT:C_Rect_L7.2mm_W5.5mm_P5.00mm_FKS2_FKP2_MKS2_MKP2 -> Capacitor_SMD:C_1206_3216Metric_Pad1.42x1.75mm_HandSolder
Connections:
- net +3V3: now also R?.2, U?.5 (VIO), U?.6 (VDD); no longer U5.3 (EN)
- net GND: now also C?.2, U?.2 (GND), U?.25 (GND)
- net at U5.35 (GPIO1/TXD0): now also U?.20 (RXD)
- net at U5.34 (GPIO3/RXD0): now also U?.21 (TXD)
- net at J1.3 (D+): now also U?.3 (D+)
- net at J1.2 (D-): now also U?.4 (D-)
- net at U5.25 (GPIO0): now also Q?.1 (C)
- net PWRON: now reaches Q?.1 (G), R?.1
- new net: Q?.3 (E), R?.2, U?.19 (RTS)
- new net: Q?.3 (E), R?.2, U?.23 (DTR)
- new net: Q?.2 (B), R?.1 (x2)
- new net RESET: C?.1, Q?.1 (C), R?.1, U5.3 (EN)
Other:
- moved on the sheet: J1

Commit message: new board improvements
Parts:
- removed Q? (x2): BC546, Package_TO_SOT_THT:TO-92_Inline, symbol Transistor_BJT:BC546
- removed Q?: IRLML2244, Package_TO_SOT_SMD:SOT-23, symbol Transistor_FET:IRLML5203
- removed R? (x2): 10k, Resistor_THT:R_Axial_DIN0204_L3.6mm_D1.6mm_P7.62mm_Horizontal, symbol Device:R
- removed R?: 100k, Resistor_THT:R_Axial_DIN0204_L3.6mm_D1.6mm_P7.62mm_Horizontal, symbol Device:R
- removed TP?: TestPoint_Batt_Switched, symbol Connector:TestPoint_Probe
- removed U1: AMS1117-1.8, Package_TO_SOT_SMD:SOT-223-3_TabPin2, symbol Regulator_Linear:AMS1117-1.8
- added C?: 10n, Capacitor_SMD:C_1206_3216Metric_Pad1.42x1.75mm_HandSolder, symbol Device:C
- added D?: RX, symbol Device:LED
- added D?: TX, symbol Device:LED
- added J?: PwrOn, symbol Connector:Conn_01x02_Male
- added Q?: DMN2020LSN, Package_TO_SOT_SMD:SOT-23, symbol Transistor_FET:DMN2056U
- added R? (x2): 10k, Resistor_THT:R_Axial_DIN0204_L3.6mm_D1.6mm_P7.62mm_Horizontal, symbol Device:R
- added R?: 100k, Resistor_THT:R_Axial_DIN0204_L3.6mm_D1.6mm_P7.62mm_Horizontal, symbol Device:R
- added R?: 1k, Resistor_THT:R_Axial_DIN0204_L3.6mm_D1.6mm_P7.62mm_Horizontal, symbol Device:R
- added R? (x2): ?, Resistor_THT:R_Axial_DIN0204_L3.6mm_D1.6mm_P7.62mm_Horizontal, symbol Device:R
- added R?: 22.1k, Resistor_THT:R_Axial_DIN0204_L3.6mm_D1.6mm_P7.62mm_Horizontal, symbol Device:R
- added R?: 47.5k, Resistor_THT:R_Axial_DIN0204_L3.6mm_D1.6mm_P7.62mm_Horizontal, symbol Device:R
- added TP?: TestPoint_EN, symbol Connector:TestPoint_Probe
- added U?: NCP115, symbol audioplayer:NCP115
- added U?: LMC555xM, Package_SO:SOIC-8_3.9x4.9mm_P1.27mm, symbol Timer:LMC555xM
- added U?: UMH4NFHA, symbol audioplayer:UMH4NFHA
- C11: value 22u -> 1u
- F?: value Fuse -> 1A
- U?: value CP2102N-A01-GQFN24 -> CP2102N-A02-GQFN24
Connections:
- net +1V8: now also U?.5 (OUT)
- net +3V3: now also U?.7 (REGIN), R?.2
- net BATT: now also C3.1, C4.1, L1.1, U2.5 (IN), U3.5 (VIN), R?.2, R?.2, R?.2, U?.1 (IN), U?.8 (VCC)
- net GND: now also C?.2, J?.2 (Pin_2), Q?.2 (S), R?.1, R?.1, R?.2, U?.1 (GND), U?.2 (GND); no longer J?.2 (Pin_2)
- net RESET: now also U?.6 (C1)
- net at C?.1, D?.2 (A), J1.1 (VBUS)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: now also R?.2
- net at U5.25 (GPIO0): now also U?.3 (C2)
- net at U?.13 (GPIO.1): now also D?.2 (A)
- net at U?.14 (GPIO.0): now also D?.2 (A)
- net at U?.19 (RTS): now also U?.1 (E1), U?.5 (B2)
- net at U?.23 (DTR): now also U?.2 (B1), U?.4 (E2)
- net at U?.8 (VBUS): now also R?.1, R?.1
- net at U?.9 (~RSTb): now also R?.1
- net at C7.1, U3.7 (PS/SYNC), U3.8 (VINA): no longer U3.6 (EN)
- net AMP_ENABLE renamed AMP_EN
- new net: J?.1 (Pin_1), R?.1, U?.2 (TR)
- new net: R?.1, U?.4 (R)
- new net: C?.1, U?.5 (CV)
- new net: Q?.1 (G), R?.1
- new net: J?.2 (Pin_2), Q?.3 (D)
- new net: D?.1 (K), R?.2 (x2)
- new net EN: TP?.1, U2.4 (EN), U3.6 (EN), U?.3 (EN), U?.3 (Q)
Other:
- note added: "CHECK FOOTPRINT!"
- note added: "Class D Stereo Amplifier"
- moved on the sheet: C11, C16, C19, C2, C20, C21, C22, C23, C4, C6, C?, D1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
