File: kicad/mainboard/audioplayer.sch (KiCad schematic (older format))
At the start: 89 parts, among them J1 USB_B, J2 Micro_SD_Card, J3 SPK, U2 MT3608, U3 TPS63031DSK, U5 ESP-WROOM32, U6 VS1053b, U7 PAM8408, Y1 12.288MHz

Commit message: new board WIP
Parts:
- removed C1, C10: 100n, Capacitor_THT:C_Disc_D5.1mm_W3.2mm_P5.00mm, symbol Device:C
- removed J3: SPK, Connector_PinHeader_2.54mm:PinHeader_1x04_P2.54mm_Vertical, symbol Connector:Conn_01x04_Male
- removed J?: PwrOn, symbol Connector:Conn_01x02_Male
- removed RN1: R_Network04, Resistor_THT:R_Array_SIP5, symbol Device:R_Network04
- removed U3: TPS63031DSK, Package_SON:WSON-10-1EP_2.5x2.5mm_P0.5mm_EP1.2x2mm, symbol Regulator_Switching:TPS63031DSK
- removed U?: NCP115, symbol audioplayer:NCP115
- added C12, C21: 100n, Capacitor_SMD:C_0603_1608Metric, symbol Device:C
- added C34, C35, C36, C37: 220p, Capacitor_SMD:C_0603_1608Metric, symbol Device:C
- added D6, D7, D8, D9: WS2812B, LED_SMD:LED_WS2812B_PLCC4_5.0x5.0mm_P3.2mm, symbol LED:WS2812B
- added J6: L, Connector_PinHeader_2.54mm:PinHeader_1x02_P2.54mm_Vertical, symbol Connector:Conn_01x02_Male
- added J7: R, Connector_PinHeader_2.54mm:PinHeader_1x02_P2.54mm_Vertical, symbol Connector:Conn_01x02_Male
- added JP1, JP2: SolderJumper_3_Bridged123, Jumper:SolderJumper-3_P1.3mm_Open_RoundedPad1.0x1.5mm_NumberLabels, symbol Jumper:SolderJumper_3_Bridged123
- added L3, L4, L5, L6: L_Core_Ferrite_Small, Inductor_SMD:L_0805_2012Metric, symbol Device:L_Core_Ferrite_Small
- added Q1: BC847, Package_TO_SOT_SMD:SOT-23, symbol Transistor_BJT:BC847
- added R1: 10k, Resistor_SMD:R_0603_1608Metric, symbol Device:R
- added R26: 100, Resistor_SMD:R_0603_1608Metric, symbol Device:R
- added R27: 220, Resistor_SMD:R_0603_1608Metric, symbol Device:R
- added SW1: LEFT, Button_Switch_THT:SW_Tactile_Straight_KSA0Axx1LFTR, symbol Switch:SW_Push
- added SW2: MID, Button_Switch_THT:SW_Tactile_Straight_KSA0Axx1LFTR, symbol Switch:SW_Push
- added SW3: RIGHT, Button_Switch_THT:SW_Tactile_Straight_KSA0Axx1LFTR, symbol Switch:SW_Push
- added SW4: VOL-, Button_Switch_THT:SW_Tactile_Straight_KSA0Axx1LFTR, symbol Switch:SW_Push
- added SW5: VOL+, Button_Switch_THT:SW_Tactile_Straight_KSA0Axx1LFTR, symbol Switch:SW_Push
- added TP7: MP3_L, TestPoint:TestPoint_Pad_D1.5mm, symbol Connector:TestPoint_Flag
- added TP8: MP3_B, TestPoint:TestPoint_Pad_D1.5mm, symbol Connector:TestPoint_Flag
- added TP9: MP3_R, TestPoint:TestPoint_Pad_D1.5mm, symbol Connector:TestPoint_Flag
- added U11: RC-552, audioplayer:RFID-RC522, symbol audioplayer:RC-552
- added U12: PC817, Package_DIP:DIP-4_W8.89mm_SMDSocket_LongPads, symbol Isolator:PC817
- added U5: NCP115, Package_SO:TSOP-5_1.65x3.05mm_P0.95mm, symbol audioplayer:NCP115
- added U7: TPS63001, Package_SON:Texas_DRC0010J_ThermalVias, symbol Regulator_Switching:TPS63001
- C1: renamed from C?; footprint Capacitor_SMD:C_1206_3216Metric_Pad1.42x1.75mm_HandSolder -> Capacitor_SMD:C_1206_3216Metric
- C10: renamed from C21; footprint Capacitor_THT:C_Disc_D5.1mm_W3.2mm_P5.00mm -> Capacitor_SMD:C_0603_1608Metric
- C11: renamed from C16; footprint Capacitor_SMD:C_1206_3216Metric_Pad1.42x1.75mm_HandSolder -> Capacitor_SMD:C_1206_3216Metric
- C13: renamed from C22; footprint Capacitor_THT:C_Disc_D5.1mm_W3.2mm_P5.00mm -> Capacitor_SMD:C_0603_1608Metric
- C14: renamed from C19; footprint Capacitor_SMD:C_1206_3216Metric_Pad1.42x1.75mm_HandSolder -> Capacitor_SMD:C_0603_1608Metric
- C15: renamed from C5; footprint Capacitor_THT:C_Disc_D5.1mm_W3.2mm_P5.00mm -> Capacitor_SMD:C_0603_1608Metric
- C16: renamed from C6; footprint Capacitor_SMD:C_1206_3216Metric_Pad1.42x1.75mm_HandSolder -> Capacitor_SMD:C_0603_1608Metric
- C17: renamed from C23; footprint Capacitor_THT:C_Disc_D5.1mm_W3.2mm_P5.00mm -> Capacitor_SMD:C_0603_1608Metric
- C18: renamed from C2; footprint (none) -> Capacitor_THT:CP_Radial_D8.0mm_P3.50mm
- C19: renamed from C9; footprint Capacitor_THT:C_Disc_D5.1mm_W3.2mm_P5.00mm -> Capacitor_SMD:C_0603_1608Metric
- C2: renamed from C?; footprint (none) -> Capacitor_SMD:C_1206_3216Metric
- C20: renamed from C8; footprint Capacitor_SMD:C_1206_3216Metric_Pad1.42x1.75mm_HandSolder -> Capacitor_SMD:C_0603_1608Metric
- C22: renamed from C13; footprint Capacitor_THT:C_Disc_D5.1mm_W3.2mm_P5.00mm -> Capacitor_SMD:C_0603_1608Metric
- C23: renamed from C24; footprint Capacitor_THT:C_Rect_L7.0mm_W2.5mm_P5.00mm -> Capacitor_SMD:C_0603_1608Metric
- C24: renamed from C25; footprint Capacitor_THT:C_Rect_L7.0mm_W2.5mm_P5.00mm -> Capacitor_SMD:C_0603_1608Metric
- C25: renamed from C15; footprint Capacitor_THT:C_Disc_D5.1mm_W3.2mm_P5.00mm -> Capacitor_SMD:C_0603_1608Metric
- C26: renamed from C17; footprint Capacitor_THT:C_Disc_D5.1mm_W3.2mm_P5.00mm -> Capacitor_SMD:C_0603_1608Metric
- C27: renamed from C18; footprint Capacitor_THT:C_Disc_D5.1mm_W3.2mm_P5.00mm -> Capacitor_SMD:C_0603_1608Metric
- C28: renamed from C26; footprint Capacitor_THT:C_Rect_L7.0mm_W2.5mm_P5.00mm -> Capacitor_SMD:C_0603_1608Metric
- C29: renamed from C27; footprint Capacitor_THT:C_Rect_L7.0mm_W2.5mm_P5.00mm -> Capacitor_SMD:C_0603_1608Metric
- C3, C4: footprint Capacitor_SMD:C_1206_3216Metric_Pad1.42x1.75mm_HandSolder -> Capacitor_SMD:C_1206_3216Metric
- C30: renamed from C28; footprint Capacitor_THT:C_Rect_L7.0mm_W2.5mm_P5.00mm -> Capacitor_SMD:C_0603_1608Metric
- C31: renamed from C29; footprint Capacitor_THT:C_Rect_L7.0mm_W2.5mm_P5.00mm -> Capacitor_SMD:C_0603_1608Metric
- C32: renamed from C30; footprint Capacitor_THT:C_Rect_L7.0mm_W2.5mm_P5.00mm -> Capacitor_SMD:C_0603_1608Metric
- C33: renamed from C31; footprint Capacitor_THT:C_Rect_L7.0mm_W2.5mm_P5.00mm -> Capacitor_SMD:C_0603_1608Metric
- C5: renamed from C7; footprint Capacitor_THT:C_Disc_D5.1mm_W3.2mm_P5.00mm -> Capacitor_SMD:C_0603_1608Metric
- C6: renamed from C11; footprint Capacitor_SMD:C_1206_3216Metric_Pad1.42x1.75mm_HandSolder -> Capacitor_SMD:C_0603_1608Metric
- C7: renamed from C?; footprint Capacitor_THT:C_Disc_D5.1mm_W3.2mm_P5.00mm -> Capacitor_SMD:C_0603_1608Metric
- C8: renamed from C12; footprint Capacitor_SMD:C_1206_3216Metric_Pad1.42x1.75mm_HandSolder -> Capacitor_SMD:C_1206_3216Metric
- C9: renamed from C20; footprint Capacitor_THT:C_Disc_D5.1mm_W3.2mm_P5.00mm -> Capacitor_SMD:C_0603_1608Metric
- D1: renamed from D?; value LED -> gn; footprint (none) -> LED_SMD:LED_0805_2012Metric
- D2: renamed from D?; value LED -> rd; footprint (none) -> LED_SMD:LED_0805_2012Metric
- D3: renamed from D?; value RX -> gn; footprint (none) -> LED_SMD:LED_0805_2012Metric
- D4: renamed from D?; value TX -> rd; footprint (none) -> LED_SMD:LED_0805_2012Metric
- D5: renamed from D1; footprint (none) -> Diode_SMD:D_SMA
- F1: renamed from F?; footprint (none) -> Fuse:Fuseholder_TR5_Littelfuse_No560_No460
- J1: footprint (none) -> Connector_USB:USB_B_Lumberg_2411_02_Horizontal
- J3: renamed from J?; footprint (none) -> Connector_PinHeader_2.54mm:PinHeader_1x02_P2.54mm_Horizontal
- J5: renamed from J2; footprint (none) -> Connector_Card:microSD_HC_Hirose_DM3AT-SF-PEJM5
- L1: footprint (none) -> Inductor_SMD:L_7.3x7.3_H4.5
- L2: value 1.5u -> 2.2u; footprint (none) -> Inductor_SMD:L_Taiyo-Yuden_NR-30xx; Type (none) -> Taiyo Yuden NR3015T1R5N
- R10, R13, R18, R2, R3, R4, R5, R6, R9: renamed from R?; footprint Resistor_THT:R_Axial_DIN0204_L3.6mm_D1.6mm_P7.62mm_Horizontal -> Resistor_SMD:R_0603_1608Metric
- R11: renamed from R?; value ? -> 270; footprint Resistor_THT:R_Axial_DIN0204_L3.6mm_D1.6mm_P7.62mm_Horizontal -> Resistor_SMD:R_0603_1608Metric
- R12: renamed from R?; value ? -> 200; footprint Resistor_THT:R_Axial_DIN0204_L3.6mm_D1.6mm_P7.62mm_Horizontal -> Resistor_SMD:R_0603_1608Metric
- R14: renamed from R3; footprint Resistor_THT:R_Axial_DIN0204_L3.6mm_D1.6mm_P7.62mm_Horizontal -> Resistor_SMD:R_0603_1608Metric
- R15: renamed from R4; footprint Resistor_THT:R_Axial_DIN0204_L3.6mm_D1.6mm_P7.62mm_Horizontal -> Resistor_SMD:R_0603_1608Metric
- R16: renamed from R2; footprint Resistor_THT:R_Axial_DIN0204_L3.6mm_D1.6mm_P7.62mm_Horizontal -> Resistor_SMD:R_0603_1608Metric
- R17: renamed from R1; footprint Resistor_THT:R_Axial_DIN0204_L3.6mm_D1.6mm_P7.62mm_Horizontal -> Resistor_SMD:R_0603_1608Metric
- R19: renamed from R6; footprint Resistor_THT:R_Axial_DIN0204_L3.6mm_D1.6mm_P7.62mm_Horizontal -> Resistor_SMD:R_0603_1608Metric
- R20: renamed from R7; footprint Resistor_THT:R_Axial_DIN0204_L3.6mm_D1.6mm_P7.62mm_Horizontal -> Resistor_SMD:R_0603_1608Metric
- R21: renamed from R10; footprint Resistor_THT:R_Axial_DIN0204_L3.6mm_D1.6mm_P7.62mm_Horizontal -> Resistor_SMD:R_0603_1608Metric
- R22: renamed from R11; footprint Resistor_THT:R_Axial_DIN0204_L3.6mm_D1.6mm_P7.62mm_Horizontal -> Resistor_SMD:R_0603_1608Metric
- R23: renamed from R8; footprint Resistor_THT:R_Axial_DIN0204_L3.6mm_D1.6mm_P7.62mm_Horizontal -> Resistor_SMD:R_0603_1608Metric
- R24: renamed from R12; footprint Resistor_THT:R_Axial_DIN0204_L3.6mm_D1.6mm_P7.62mm_Horizontal -> Resistor_SMD:R_0603_1608Metric
- R25: renamed from R9; value 22k -> 10k; footprint Resistor_THT:R_Axial_DIN0204_L3.6mm_D1.6mm_P7.62mm_Horizontal -> Resistor_SMD:R_0603_1608Metric
- R7: renamed from R?; value 1k -> 10k; footprint Resistor_THT:R_Axial_DIN0204_L3.6mm_D1.6mm_P7.62mm_Horizontal -> Resistor_SMD:R_0603_1608Metric
- R8: renamed from R5; footprint Resistor_THT:R_Axial_DIN0204_L3.6mm_D1.6mm_P7.62mm_Horizontal -> Resistor_SMD:R_0603_1608Metric
- TP1, TP2, TP3, TP4, TP5, TP6: renamed from TP?; footprint (none) -> TestPoint:TestPoint_Pad_D1.5mm
- U10: renamed from U7; footprint (none) -> Package_SO:SO-16_5.3x10.2mm_P1.27mm
- U4: renamed from U?; value UMH4NFHA -> UMH4NTN; footprint (none) -> Package_TO_SOT_SMD:SOT-363_SC-70-6
- U8: renamed from U5; footprint (none) -> audioplayer:ESP32-WROOM
- U9: renamed from U6; footprint (none) -> Package_QFP:LQFP-48_7x7mm_P0.5mm
- Y1: footprint (none) -> Crystal:Crystal_SMD_HC49-SD
- gave numbers to parts that had none: 4
- renumbered U2 to U6
Connections:
- net +1V8: now also U5.5 (OUT)
- net +3V3: now also C12.1, C21.1, D6.1 (VDD), D7.1 (VDD), D8.1 (VDD), D9.1 (VDD), U11.8 (+3.3V), U7.1 (VOUT), U7.10 (FB)
- net BATT: now also R26.2, R27.2, U5.1 (IN), U7.5 (VIN)
- net EN: now also U5.3 (EN), U7.6 (EN)
- net GND: now also R10.1, C12.2, C21.2, C34.2, C35.1, C36.2, C37.1, D6.3 (VSS), D7.3 (VSS), D8.3 (VSS), D9.3 (VSS), Q1.2 (E), SW1.1, SW2.1, SW3.2, SW4.2, SW5.2, U11.6 (GND), U12.3, U5.2 (GND), U7.11 (PGND), U7.3 (PGND), U7.9 (GND); no longer D2.1 (K)
- net MISO: now also U11.4 (MISO)
- net MOSI: now also U11.3 (MOSI)
- net RFID_CS: now also U11.1 (SS)
- net RFID_RST: now also U11.7 (RST)
- net SCK: now also U11.2 (SCK)
- net at U10.10 (LOUTP): now also L3.1
- net at U10.11 (LOUTN): now also L4.2
- net at U10.15 (ROUTP): now also L5.1
- net at U10.14 (ROUTN): now also L6.2
- net at R22.2, R23.2, U9.46 (LEFT): now also TP7.1
- net at R21.2, R24.2, U9.39 (RIGHT): now also TP9.1
- net at R20.2, U10.1 (RINP), U10.8 (LINP)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: now also TP8.1
- net at C2.1, J1.1 (VBUS), R2.2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: now also R9.2; no longer D1.2 (A)
- net at U8.33 (GPIO21): now also JP2.1 (A)
- net ESPRXD: now reaches U3.21 (TXD), U8.34 (GPIO3/RXD0)
- net ESPTXD: now reaches U3.20 (RXD), U8.35 (GPIO1/TXD0)
- net at U8.36 (GPIO22): now also JP1.1 (A)
- net at D2.2 (A): now also D1.1 (K), U2.1 (STAT); no longer R10.1
- net at R5.1, U1.2 (TR): now also U12.4
- net at R3.1, U1.4 (R): now also Q1.3 (C)
- net at L2.2: now also U7.2 (L2)
- net at L2.1: now also U7.4 (L1)
- net at C5.1: now also R26.1, U7.7 (PS/SYNC), U7.8 (VINA)
- net LED1 renamed WS2812
- net WS2812: now also D6.4 (DIN)
- net LED2 renamed PWR_DOWN
- net PWR_DOWN: now also R1.1
- net LED3: no longer names the net of U8.13 (GPIO14)
- net LED4: no longer names the net of U8.14 (GPIO12)
- net SW1: no longer names the net of U8.5 (SENSOR_VN/GPIO39)
- net SW1: now also SW1.2
- net SW2 renamed PWR_UP
- net PWR_UP: now also SW2.2, U12.2
- net SW3: no longer names the net of U8.7 (GPIO35)
- net SW3: now also SW3.1
- net SW4: no longer names the net of U8.6 (GPIO34)
- net VOL+ renamed AMP_VOL+
- net AMP_VOL+: now also JP2.2 (C)
- net VOL- renamed AMP_VOL-
- net AMP_VOL-: now also JP1.2 (C)
- new net: D2.1 (K), R10.2
- new net: D1.2 (A), R9.1
- new net: JP1.3 (B), SW4.1
- new net: JP2.3 (B), SW5.1
- new net: R27.1, U12.1
- new net: D6.2 (DOUT), D7.4 (DIN)
- new net: D7.2 (DOUT), D8.4 (DIN)
- new net: D8.2 (DOUT), D9.4 (DIN)
- new net: Q1.1 (B), R1.2
- new net: C36.1, J6.1 (Pin_1), L4.1
- new net: C34.1, J6.2 (Pin_2), L3.2
- new net: C37.2, J7.2 (Pin_2), L5.2
- new net: C35.2, J7.1 (Pin_1), L6.1
Other:
- moved on the sheet: C1, C20, C23, C24, C28, C29, C3, C30, C31, C32, C33, D1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

Commit message: new board WIP
Parts:
- added C?: 100n, Capacitor_SMD:C_0603_1608Metric, symbol Device:C
Connections:
- net +3V3: now also C?.1
- net GND: now also C?.2
Changed lines of the file:
@@
 Wire Wire Line
 	8800 6900 8575 6900
-Wire Bus Line
-	8475 1000 8475 4600
 Wire Wire Line
 	8575 7275 8575 7250
@@
 	1    0    0    -1
 $EndComp
+$Comp
+L Device:C C?
+U 1 1 5F2FDB6F
+P 9300 10750
+F 0 "C?" H 9415 10796 50  0000 L CNN
+F 1 "100n" H 9415 10705 50  0000 L CNN
+F 2 "Capacitor_SMD:C_0603_1608Metric" H 9338 10600 50  0001 C CNN
+F 3 "~" H 9300 10750 50  0001 C CNN
+	1    9300 10750
+	1    0    0    -1
+$EndComp
+Wire Wire Line
+	8875 10500 9300 10500
+Wire Wire Line
+	9300 10500 9300 10600
+Connection ~ 8875 10500
+Wire Wire Line
+	9300 10950 8875 10950
+Wire Wire Line
+	9300 10900 9300 10950
+Wire Bus Line
+	8475 1000 8475 4600
+Connection ~ 8875 10950
 $EndSCHEMATC
