File: kicad/mainboard/audioplayer.sch (KiCad schematic (older format))
At the start: 117 parts, among them J1 USB_B, J3 LiPo, J5 Micro_SD_Card, J6 L, J7 R, Q1 BC847, Q2 DMN2020LSN, SW1 LEFT, SW2 MID, SW3 RIGHT, SW4 VOL-, SW5 VOL+, U1 LMC555xM, U10 PAM8408, U11 RC-552, U12 PC817, U2 MCP73831-2-OT, U3 CP2102N-A02-GQFN24, U4 UMH4NTN, U5 NCP115, U6 MT3608, U7 TPS63001, U8 ESP-WROOM32, U9 VS1053b, Y1 12.288MHz

Commit message: new board BOM consoldifation
Parts:
- removed R11: 270, Resistor_SMD:R_0603_1608Metric, symbol Device:R
- added R12, R16: 1k, Resistor_SMD:R_0603_1608Metric, symbol Device:R
- added R20: 20, Resistor_SMD:R_0603_1608Metric, symbol Device:R
- added R28: 100k, Resistor_SMD:R_0603_1608Metric, symbol Device:R
- added R30, R5, R7, R8, R9: 100, Resistor_SMD:R_0603_1608Metric, symbol Device:R
- C1: renamed from C7; Type (none) -> X5R
- C10: renamed from C6; Type (none) -> X7R
- C11: renamed from C9; Type (none) -> X5R
- C12: renamed from C10; Type (none) -> X5R
- C13: Type (none) -> X5R
- C14: renamed from C17; Type (none) -> X5R
- C15: renamed from C28; Type (none) -> X7R
- C2: renamed from C20; Type (none) -> X7R
- C21: renamed from C4; Type (none) -> X7R
- C22: renamed from C11; Type (none) -> X7R
- C23: renamed from C14; Type (none) -> X7R
- C24: renamed from C16; Type (none) -> X7R
- C25: renamed from C18; Type (none) -> Electrolytic; Vorrätig (none) -> ok
- C26: renamed from C8; Type (none) -> X7R
- C27: renamed from C1; footprint Capacitor_SMD:C_1206_3216Metric -> Capacitor_SMD:C_0603_1608Metric
- C28: renamed from C3; value 10u -> 22u; Type (none) -> X7R
- C29: renamed from C5; Type (none) -> X5R
- C3: renamed from C2; value 10u -> 22u; Type (none) -> X7R
- C30: renamed from C12; Type (none) -> X5R
- C31: renamed from C15; Type (none) -> X5R
- C32: renamed from C19; Type (none) -> X5R
- C33: renamed from C21; Type (none) -> X5R
- C34: renamed from C22; Type (none) -> X5R
- C35: renamed from C25; Type (none) -> X5R
- C36: renamed from C26; Type (none) -> X5R
- C37: renamed from C27; Type (none) -> X5R
- C38: renamed from C?; Type (none) -> X5R
- D5: renamed from D3; value gn -> green; Farnell (none) -> 1318243
- D6: renamed from D4; value rd -> red; Farnell (none) -> 1318244
- D7: renamed from D1; value gn -> green; Farnell (none) -> 1318243
- D8: renamed from D2; value rd -> red; Farnell (none) -> 1318244
- F1: value 1A -> 1A F; Vorrätig (none) -> ok
- J1: renamed from J5; Farnell (none) -> 1764374
- J3: renamed from J6; Vorrätig (none) -> ok
- J4: renamed from J7; Vorrätig (none) -> ok
- J5: renamed from J3; Vorrätig (none) -> ok
- JP1: renamed from JP2; Vorrätig (none) -> ok
- JP2: renamed from JP1; Vorrätig (none) -> ok
- R13: renamed from R9; value 470 -> 1k
- R14: renamed from R8; value 2k -> 1k
- R21: renamed from R20; value 10 -> 20
- R27: renamed from R14; value 47k -> 100k
- R31: renamed from R27; value 220 -> 100
- R6: renamed from R12; value 200 -> 100
- SW1: renamed from SW4; Info (none) -> VOL-
- SW2: renamed from SW5; Info (none) -> LEFT
- SW3: Info (none) -> MID
- SW5: renamed from SW2; Info (none) -> VOL+
- TP1: renamed from TP7; Vorrätig (none) -> ok
- TP2: renamed from TP9; Vorrätig (none) -> ok
- TP3: renamed from TP8; Vorrätig (none) -> ok
- TP4: Vorrätig (none) -> ok
- TP5: renamed from TP1; Vorrätig (none) -> ok
- TP6: renamed from TP2; Vorrätig (none) -> ok
- TP7: renamed from TP6; Vorrätig (none) -> ok
- TP8: renamed from TP3; Vorrätig (none) -> ok
- TP9: renamed from TP5; Vorrätig (none) -> ok
- renumbered C29 to C16, C30 to C17, C31 to C18, C32 to C19, C33 to C20, C23 to C4, C34 to C5, C36 to C6, C24 to C7, C35 to C8, C37 to C9, D6 to D1, D7 to D2, D8 to D3, D9 to D4, D5 to D9, J1 to J2, L3 to L1, L4 to L2, L5 to L3, L6 to L4, L1 to L5, L2 to L6, Q2 to Q1, Q1 to Q2, R13 to R1, R16 to R10, R17 to R11, R10 to R15, R18 to R17, R23 to R18, R24 to R19, R7 to R2, R21 to R22, R22 to R23, R19 to R24, R6 to R26, R15 to R29, R2 to R3, R3 to R32, R5 to R33, R26 to R34, R1 to R35, SW1 to SW4, U11 to U1, U12 to U10, U1 to U11, U7 to U12, U4 to U2, U8 to U3, U3 to U4, U2 to U5, U10 to U6, U9 to U7, U5 to U8, U6 to U9
Connections:
- wire segments 516 -> 537
Other:
- note removed: "X7R"
- moved on the sheet: C22, C24, C3, D7, D8, D9, R13, R14, R15, R27, R31, R6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

Commit message: board layout finalization
Parts:
- added R29: 2.7k, Resistor_SMD:R_0603_1608Metric, symbol Device:R
- C1, C11, C12, C13, C14, C29, C30, C31, C32, C33, C34, C35, C36, C37, C38, R1, R10, R11, R12, R13, R14, R15, R16, R17, R18, R19, R2, R20, R21, R22, R23, R24, R25, R26, R27, R28, R5, R6, R7, R8, R9: Vorrätig (none) -> ok
- C10, C15, C2, C23, C24: value 1u -> 1u 10V; footprint Capacitor_SMD:C_0603_1608Metric -> Capacitor_SMD:C_0805_2012Metric; Mouser (none) -> 963-EMK212B7105KG-T; Vorrätig (none) -> ok
- C16: footprint Capacitor_SMD:C_0603_1608Metric -> Capacitor_SMD:C_0805_2012Metric; Mouser (none) -> 80-C0805C473J3GEAULR; Type (none) -> C0G
- C17, C18, C27: Mouser (none) -> 81-GRM1885C1E103JA1D; Type (none) -> C0G
- C19, C20: Farnell (none) -> 2906783; Mouser (none) -> 810-CGA3E2C0G1H472J; Type (none) -> C0G
- C21, C26, C28, C3: value 22u -> 22u 10V; footprint Capacitor_SMD:C_1206_3216Metric -> Capacitor_SMD:C_1210_3225Metric; Mouser (none) -> 963-EMK325B7226MMHP
- C22: footprint Capacitor_SMD:C_1206_3216Metric -> Capacitor_SMD:C_1210_3225Metric; Mouser (none) -> 963-EMK325B7226MMHP
- C4, C7: Type (none) -> C0G; Vorrätig (none) -> ok
- C5, C6, C8, C9: Type (none) -> X7R; Vorrätig (none) -> ok
- D1, D2, D3, D4: aliexpress (none) -> OK
- D5, D7: Mouser (none) -> 710-150080VS75000
- D6, D8: Mouser (none) -> 710-150080RS75000
- D9: Farnell (none) -> 2211964; Mouser (none) -> 652-CD214A-F150
- J1: Mouser (none) -> 798-DM3AT-SF-PEJM5
- J2: Farnell (none) -> 1308876; Mouser (none) -> 490-UJ2-BH-1-TH; Vorrätig (none) -> ok
- L1, L2, L3, L4: value L_Core_Ferrite_Small -> 600; Farnell (none) -> 1635719; Mouser (none) -> 710-74279204
- L5: value 10u -> 22u; footprint Inductor_SMD:L_7.3x7.3_H4.5 -> Inductor_SMD:L_Taiyo-Yuden_NR-60xx; Mouser (none) -> 963-NR6028T220M
- L6: Mouser (none) -> 963-NR6028T2R2N; Type Taiyo Yuden NR3015T1R5N -> (none)
- Q1: footprint Package_TO_SOT_SMD:SOT-23 -> Package_TO_SOT_SMD:SC-59; Farnell (none) -> 2543536; Mouser (none) -> 621-DMN2020LSN-7
- Q2: Farnell (none) -> 1081230; Mouser (none) -> 863-BC847BLT1G
- R3: Mouser (none) -> 71-CRCW120622K1FKEAC
- R30: renamed from R29; value 5.6k -> 2.7k; Vorrätig (none) -> ok
- R31: renamed from R30; Vorrätig (none) -> ok
- R32: renamed from R31; Vorrätig (none) -> ok
- R33: renamed from R32; Vorrätig (none) -> ok
- R34: renamed from R33; Vorrätig (none) -> ok
- R35: renamed from R34; Vorrätig (none) -> ok
- R36: renamed from R35; Vorrätig (none) -> ok
- R4: footprint Resistor_SMD:R_0603_1608Metric -> Resistor_SMD:R_1206_3216Metric; Mouser (none) -> 71-CRCW120647K5FKEAC
- SW1, SW2, SW3, SW4, SW5: Farnell (none) -> 2468761
- U1, U3, U7, U9: Farnell (none) -> -; aliexpress (none) -> OK
- U10: Farnell (none) -> -; Mouser (none) -> 852-PC81710NIP1B
- U11: footprint Package_SO:SOIC-8_3.9x4.9mm_P1.27mm -> Package_SO:VSSOP-8_3.0x3.0mm_P0.65mm; Mouser (none) -> 926-LMC555CMMX/NOPB
- U12: Farnell (none) -> 3008242; Mouser (none) -> 595-TPS63001DRCR
- U2: Farnell (none) -> 1680405; Mouser (none) -> 755-UMH4NTN
- U4: Farnell (none) -> -; Mouser (none) -> 634-CP2102NA02GQFN24
- U5: Farnell (none) -> 1332158; Mouser (none) -> 579-MCP73832T2DFI/OT
- U6: Farnell (none) -> -; Mouser (none) -> 621-PAM8408DR
- U8: Farnell (none) -> 2981135; Mouser (none) -> 863-NCP115ASN180T1G
- Y1: Farnell (none) -> 3228382; Mouser (none) -> 815-ABLS12288MHZD3YT
Connections:
- wire segments 537 -> 540
Other:
- note removed: "CHECK FOOTPRINT!"
- moved on the sheet: R30

Commit message: board polish
Connections:
- net labels added: AMP_PWR_EN
- wire segments 540 -> 541
Other:
- moved on the sheet: JP2
Changed lines of the file:
@@
 L Jumper:SolderJumper_3_Bridged123 JP2
 U 1 1 628BA939
-P 7425 3250
-F 0 "JP2" H 7375 3400 50  0000 L CNN
-F 1 "SolderJumper_3_Bridged123" H 7425 3454 50  0001 C CNN
-F 2 "Jumper:SolderJumper-3_P1.3mm_Open_RoundedPad1.0x1.5mm_NumberLabels" H 7425 3250 50  0001 C CNN
-F 3 "~" H 7425 3250 50  0001 C CNN
-F 4 "ok" H 7425 3250 50  0001 C CNN "Vorrätig"
-	1    7425 3250
-	1    0    0    -1
-$EndComp
-Wire Wire Line
-	7625 3250 8175 3250
-Wire Wire Line
-	6650 3250 7225 3250
-Text GLabel 7425 3450 3    50   Input ~ 0
+P 7575 3250
+F 0 "JP2" H 7525 3400 50  0000 L CNN
+F 1 "SolderJumper_3_Bridged123" H 7575 3454 50  0001 C CNN
+F 2 "Jumper:SolderJumper-3_P1.3mm_Open_RoundedPad1.0x1.5mm_NumberLabels" H 7575 3250 50  0001 C CNN
+F 3 "~" H 7575 3250 50  0001 C CNN
+F 4 "ok" H 7575 3250 50  0001 C CNN "Vorrätig"
+	1    7575 3250
+	1    0    0    -1
+$EndComp
+Wire Wire Line
+	7775 3250 8175 3250
+Wire Wire Line
+	6650 3250 7375 3250
+Text GLabel 7575 3450 3    50   Input ~ 0
 AMP_VOL-
 Wire Wire Line
-	7425 3450 7425 3400
+	7575 3450 7575 3400
 Text GLabel 675  10675 3    50   Input ~ 0
 PWR_DOWN
@@
 Wire Wire Line
 	4775 8800 4775 8525
-Wire Bus Line
-	8475 1000 8475 4600
 Connection ~ 4775 8525
 Wire Wire Line
@@
 	1    0    0    -1
 $EndComp
+Text GLabel 6900 3850 2    50   Input ~ 0
+AMP_PWR_EN
+Wire Wire Line
+	6650 3850 6900 3850
+Wire Bus Line
+	8475 1000 8475 4600
 $EndSCHEMATC

Commit message: use zener diode array
Parts:
- removed Q2: BC847, Package_TO_SOT_SMD:SOT-23, symbol Transistor_BJT:BC847
- removed R31, R32: 100, Resistor_SMD:R_0603_1608Metric, symbol Device:R
- removed R36: 10k, Resistor_SMD:R_0603_1608Metric, symbol Device:R
- removed U10: PC817, Package_DIP:DIP-4_W8.89mm_SMDSocket_LongPads, symbol Isolator:PC817
- added D10: 3.3V, Package_TO_SOT_SMD:SOT-23, symbol Diode:MMBZxx
- C10: renamed from C15; value 1u 10V -> 1u
- C16: renamed from C21; value 22u 10V -> 22u
- C18: renamed from C23; value 1u 10V -> 1u
- C19: renamed from C24; value 1u 10V -> 1u
- C2: value 1u 10V -> 1u
- C21: renamed from C10; value 1u 10V -> 1u
- C27: renamed from C26; value 22u 10V -> 22u
- C28, C3: value 22u 10V -> 22u
- Y1: Mouser 815-ABLS12288MHZD3YT -> ABLS7M-12.288MHZ-B-2-T
- renumbered C16 to C11, C17 to C12, C18 to C13, C19 to C14, C20 to C15, C22 to C17, C25 to C20, C11 to C22, C12 to C23, C13 to C24, C14 to C25, C27 to C26, R12 to R11, R13 to R12, R11 to R13, R26 to R20, R20 to R21, R21 to R22, R22 to R23, R23 to R24, R24 to R25, R25 to R26, R33 to R31, R34 to R32, R35 to R33, SW3 to SW1, SW1 to SW2, SW2 to SW3, TP5 to TP4, TP6 to TP5, TP7 to TP6, TP4 to TP7, U11 to U10, U12 to U11, U9 to U8, U8 to U9
Connections:
- net labels removed: AMP_PWR_EN
- wire segments 541 -> 528
Other:
- moved on the sheet: C16, C17, C18, C19, C2, C20, C21, C22, C23, C24, C25, C26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

Commit message: new board v1
Parts:
- removed R28: 100k, Resistor_SMD:R_0603_1608Metric, symbol Device:R
- removed R29: 2.7k, Resistor_SMD:R_0603_1608Metric, symbol Device:R
- added C23, C24: 100n, Capacitor_SMD:C_0603_1608Metric, symbol Device:C
- added R30: 20k, Resistor_SMD:R_0603_1608Metric, symbol Device:R
- F1: footprint Fuse:Fuseholder_TR5_Littelfuse_No560_No460 -> Fuse:Fuse_Littelfuse_372_D8.50mm
- L6: footprint Inductor_SMD:L_Taiyo-Yuden_NR-30xx -> Inductor_SMD:L_Taiyo-Yuden_NR-60xx
- R3: footprint Resistor_SMD:R_0603_1608Metric -> Resistor_SMD:R_1206_3216Metric
- R31: renamed from R30; value 2.7k -> 27k
- TP6: value TestPoint_5V5 -> TestPoint_5V3
- Y1: footprint Crystal:Crystal_SMD_HC49-SD -> audioplayer:Crystal_SMD_ABLS7M
- renumbered C33 to C21, C30 to C22, C21 to C25, C22 to C26, C23 to C27, C24 to C28, C25 to C29, C26 to C30, C27 to C31, C28 to C32, C29 to C33, C31 to C34, C32 to C35, C34 to C36, C35 to C37, C36 to C38, C37 to C39, C38 to C40, D5 to D1, D6 to D2, D7 to D3, D8 to D4, D1 to D5, D2 to D6, D3 to D7, D4 to D8, R31 to R28, R32 to R29, R33 to R32, TP8 to TP7, TP7 to TP8, U9 to U10, U10 to U9
Connections:
- net +3V3: no longer C21.1, C22.1, D5.1 (VDD), D6.1 (VDD), D7.1 (VDD), D8.1 (VDD)
- net +6V: now also C21.1, C22.1, D5.1 (VDD), D6.1 (VDD), D7.1 (VDD), D8.1 (VDD), C23.1, C24.1
- net GND: now also C23.2, C24.2, R30.2
- net at R27.1, U8.3 (FB): now also R31.1, R30.1
Other:
- note added: "6V Supply (Step Up) (Nominal 5.3V)"
- note removed: "6V Supply (Step Up)"
- moved on the sheet: C16, C17, C18, C19, C20, C21, C22, C25, C26, C27, C28, C29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

Commit message: new board software first step
Parts:
- added C41: 100n, Capacitor_SMD:C_0603_1608Metric, symbol Device:C
- added D11, D12: US1A, Diode_SMD:D_SMA, symbol Diode:US1A
- added Q2: SSM3J332R, Package_TO_SOT_SMD:SOT-23, symbol Transistor_FET:DMG2301L
- added Q3: BC547, Package_TO_SOT_SMD:SOT-23, symbol Transistor_BJT:BC547
- added R33: 1k, Resistor_SMD:R_0603_1608Metric, symbol Device:R
- added R34: 10k, Resistor_SMD:R_0603_1608Metric, symbol Device:R
- added R35: 220k, Resistor_SMD:R_0603_1608Metric, symbol Device:R
Connections:
- net +6V: now also D11.2 (A); no longer C21.1, C22.1, C23.1, C24.1, D5.1 (VDD), D6.1 (VDD), D7.1 (VDD), D8.1 (VDD)
- net BATT: now also Q2.3 (D), R33.1; no longer C16.1, C32.1, L5.1, R10.2, R32.2, U10.1 (IN), U11.5 (VIN), U8.5 (IN)
- net EN: now also R34.2; no longer U10.3 (EN), U11.6 (EN), U8.4 (EN)
- net GND: now also Q3.3 (E)
- net PWR_DOWN: now also C41.2, R35.1; no longer D10.1 (K), R28.1, U9.4 (R)
- net at C33.1, R32.1, U11.7 (PS/SYNC)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: now also U11.6 (EN)
- new net: Q2.1 (G), Q3.1 (C), R33.2
- new net: D11.1 (K), D12.2 (A)
- new net: C41.1, D10.1 (K), R28.1, R35.2, U9.4 (R)
- new net: Q3.2 (B), R34.1
- new net +4V: C21.1, C22.1, C23.1, C24.1, D12.1 (K), D5.1 (VDD), D6.1 (VDD), D7.1 (VDD), D8.1 (VDD)
- new net BATT_SWITCHED: C16.1, C32.1, L5.1, Q2.2 (S), R10.2, R32.2, U10.1 (IN), U10.3 (EN), U11.5 (VIN), U8.4 (EN), U8.5 (IN)
Other:
- note added: "6V Supply (Step Up) (Nominal 5.7V)"
- note removed: "6V Supply (Step Up) (Nominal 5.3V)"
- moved on the sheet: C16, C17, C18, C19, C20, C21, C22, C23, C24, C31, C32, C33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
