File: kicad/mainboard/audioplayer.sch (KiCad schematic (older format))
At the start: 141 parts, among them IC1 XC6193BANNER-G, J1 Micro_SD_Card, J2 USB_B, J3 L, J4 R, Q1 DMN2020LSN, Q2 SSM3J332R, SW1 RIGHT, SW2 VOL-, SW3 VOL+, SW4 LEFT, SW5 MID, U1 RC-552, U10 NCP115, U11 TPS63001, U2 UMH4NTN, U3 ESP-WROOM32, U4 CP2102N-A02-GQFN24, U5 MCP73831-2-OT, U6 PAM8408, U7 VS1053b, U8 MT3608, Y1 12.288MHz

Commit message: v2 rev2
Parts:
- added D12: US1A, Diode_SMD:D_SMA, symbol Diode:US1A
- added J5: CHG, Connector_PinHeader_2.54mm:PinHeader_1x02_P2.54mm_Vertical, symbol Connector:Conn_01x02_Male
- J2: symbol Connector:USB_B -> audioplayer-rescue:USB_B-Connector
- JP5: value PS_6V -> P_6V
- TP1: value MP3_L -> L
- TP2: value MP3_R -> R
- TP3: value MP3_B -> B
- renumbered SW2 to SW1, SW4 to SW2, SW5 to SW3, SW1 to SW4, SW3 to SW5
Connections:
- net GND: now also J5.1 (Pin_1)
- net VBUS: now also J5.2 (Pin_2)
- net at D11.1 (K): now also D12.2 (A); no longer JP4.1 (A)
- new net: D12.1 (K), JP4.1 (A)
Other:
- moved on the sheet: D11, TP14, TP9
Changed lines of the file:
@@
 	3100 2125 5250 2125
 $Comp
-L Connector:USB_B J2
+L audioplayer-rescue:USB_B-Connector J2
 U 1 1 5F43C859
 P 900 2825
@@
 ESPRXD
 $Comp
-L Switch:SW_Push SW4
+L Switch:SW_Push SW2
 U 1 1 5F2C98E2
 P 4400 3700
-F 0 "SW4" V 4446 3848 50  0000 L CNN
+F 0 "SW2" V 4446 3848 50  0000 L CNN
 F 1 "LEFT" V 4355 3848 50  0000 L CNN
 F 2 "Button_Switch_THT:SW_Tactile_Straight_KSA0Axx1LFTR" H 4400 3900 50  0001 C CNN
@@
 $EndComp
 $Comp
-L Switch:SW_Push SW1
+L Switch:SW_Push SW4
 U 1 1 5F2CDE37
 P 5175 3700
-F 0 "SW1" V 5129 3848 50  0000 L CNN
+F 0 "SW4" V 5129 3848 50  0000 L CNN
 F 1 "RIGHT" V 5220 3848 50  0000 L CNN
 F 2 "Button_Switch_THT:SW_Tactile_Straight_KSA0Axx1LFTR" H 5175 3900 50  0001 C CNN
@@
 $EndComp
 $Comp
-L Switch:SW_Push SW2
+L Switch:SW_Push SW1
 U 1 1 5F45AA3C
 P 7650 3700
-F 0 "SW2" V 7604 3848 50  0000 L CNN
+F 0 "SW1" V 7604 3848 50  0000 L CNN
 F 1 "VOL-" V 7695 3848 50  0000 L CNN
 F 2 "Button_Switch_THT:SW_Tactile_Straight_KSA0Axx1LFTR" H 7650 3900 50  0001 C CNN
@@
 $EndComp
 $Comp
-L Switch:SW_Push SW3
+L Switch:SW_Push SW5
 U 1 1 5F45B63C
 P 8075 3700
-F 0 "SW3" V 8029 3848 50  0000 L CNN
+F 0 "SW5" V 8029 3848 50  0000 L CNN
 F 1 "VOL+" V 8120 3848 50  0000 L CNN
 F 2 "Button_Switch_THT:SW_Tactile_Straight_KSA0Axx1LFTR" H 8075 3900 50  0001 C CNN
@@
 PWR_UP
 $Comp
-L Switch:SW_Push SW5
+L Switch:SW_Push SW3
 U 1 1 6094EAD1
 P 4825 3700
-F 0 "SW5" V 4871 3848 50  0000 L CNN
+F 0 "SW3" V 4871 3848 50  0000 L CNN
 F 1 "MID" V 4780 3848 50  0000 L CNN
 F 2 "Button_Switch_THT:SW_Tactile_Straight_KSA0Axx1LFTR" H 4825 3900 50  0001 C CNN
@@
 P 10550 6400
 F 0 "TP1" H 10810 6494 50  0000 L CNN
-F 1 "MP3_L" H 10810 6403 50  0000 L CNN
+F 1 "L" H 10810 6403 50  0000 L CNN
 F 2 "TestPoint:TestPoint_Pad_D1.5mm" H 10750 6400 50  0001 C CNN
 F 3 "~" H 10750 6400 50  0001 C CNN
@@
 P 11125 6400
 F 0 "TP2" H 11385 6494 50  0000 L CNN
-F 1 "MP3_R" H 11385 6403 50  0000 L CNN
+F 1 "R" H 11385 6403 50  0000 L CNN
 F 2 "TestPoint:TestPoint_Pad_D1.5mm" H 11325 6400 50  0001 C CNN
 F 3 "~" H 11325 6400 50  0001 C CNN
@@
 P 10775 6825
 F 0 "TP3" H 11035 6919 50  0000 L CNN
-F 1 "MP3_B" H 11035 6828 50  0000 L CNN
+F 1 "B" H 11035 6828 50  0000 L CNN
 F 2 "TestPoint:TestPoint_Pad_D1.5mm" H 10975 6825 50  0001 C CNN
 F 3 "~" H 10975 6825 50  0001 C CNN
@@
 	1200 2625 1325 2625
 Connection ~ 1325 2625
-Wire Wire Line
-	1325 3700 1325 2625
 Text GLabel 1275 8275 0    50   Input ~ 0
 PWR_UP
@@
 L power:+6V #PWR028
 U 1 1 5FC4A8CB
-P 12375 1200
-F 0 "#PWR028" H 12375 1050 50  0001 C CNN
-F 1 "+6V" H 12390 1373 50  0000 C CNN
-F 2 "" H 12375 1200 50  0001 C CNN
-F 3 "" H 12375 1200 50  0001 C CNN
-	1    12375 1200
+P 12075 1200
+F 0 "#PWR028" H 12075 1050 50  0001 C CNN
+F 1 "+6V" H 12090 1373 50  0000 C CNN
+F 2 "" H 12075 1200 50  0001 C CNN
+F 3 "" H 12075 1200 50  0001 C CNN
+	1    12075 1200
 	1    0    0    -1
 $EndComp
@@
 L Connector:TestPoint_Probe TP9
 U 1 1 60B760F6
-P 7125 10100
-F 0 "TP9" H 7275 10250 50  0000 L CNN
-F 1 "3.3V" H 7275 10175 50  0000 L CNN
-F 2 "TestPoint:TestPoint_Pad_D1.5mm" H 7325 10100 50  0001 C CNN
-F 3 "~" H 7325 10100 50  0001 C CNN
-F 4 "ok" H 7125 10100 50  0001 C CNN "Vorrätig"
-	1    7125 10100
+P 6775 10100
+F 0 "TP9" H 6925 10250 50  0000 L CNN
+F 1 "3.3V" H 6925 10175 50  0000 L CNN
+F 2 "TestPoint:TestPoint_Pad_D1.5mm" H 6975 10100 50  0001 C CNN
+F 3 "~" H 6975 10100 50  0001 C CNN
+F 4 "ok" H 6775 10100 50  0001 C CNN "Vorrätig"
+	1    6775 10100
 	1    0    0    -1
 $EndComp
@@
 	1    0    0    -1
 $EndComp
-Wire Wire Line
-	6975 10100 6975 10200
-Wire Wire Line
-	6975 10500 6975 10550
 Text GLabel 6050 4025 0    50   Input ~ 0
 BATT_SWITCHED
@@
 L Diode:US1A D11
 U 1 1 5F79F03F
-P 12575 1300
-F 0 "D11" H 12575 1083 50  0000 C CNN
-F 1 "US1A" H 12575 1174 50  0000 C CNN
-F 2 "Diode_SMD:D_SMA" H 12575 1125 50  0001 C CNN
-F 3 "https://www.diodes.com/assets/Datasheets/ds16008.pdf" H 12575 1300 50  0001 C CNN
-	1    12575 1300
+P 12275 1300
+F 0 "D11" H 12275 1083 50  0000 C CNN
+F 1 "US1A" H 12275 1174 50  0000 C CNN
+F 2 "Diode_SMD:D_SMA" H 12275 1125 50  0001 C CNN
+F 3 "https://www.diodes.com/assets/Datasheets/ds16008.pdf" H 12275 1300 50  0001 C CNN
+	1    12275 1300
 	-1   0    0    1
 $EndComp
@@
 $EndComp
 Wire Wire Line
-	12425 1300 12375 1300
+	12125 1300 12075 1300
 Wire Wire Line
-	12375 1300 12375 1200
+	12075 1300 12075 1200
 $Comp
 L Jumper:Jumper_2_Open JP7
@@
 Wire Wire Line
 	4575 9700 4500 9700
-Wire Wire Line
-	12725 1300 12750 1300
 $Comp
 L Jumper:Jumper_2_Open JP5
@@
 P 4700 7950
 F 0 "JP5" H 4700 8185 50  0000 C CNN
-F 1 "PS_6V" H 4700 8094 50  0000 C CNN
+F 1 "P_6V" H 4700 8094 50  0000 C CNN
 F 2 "Jumper:SolderJumper-2_P1.3mm_Open_RoundedPad1.0x1.5mm" H 4700 7950 50  0001 C CNN
 F 3 "~" H 4700 7950 50  0001 C CNN
@@
 L Connector:TestPoint_Probe TP14
 U 1 1 628518F7
-P 7125 10550
-F 0 "TP14" V 7300 10550 50  0000 L CNN
-F 1 "GND" V 7375 10550 50  0000 L CNN
-F 2 "TestPoint:TestPoint_Pad_D1.5mm" H 7325 10550 50  0001 C CNN
-F 3 "~" H 7325 10550 50  0001 C CNN
-F 4 "ok" H 7125 10550 50  0001 C CNN "Vorrätig"
-	1    7125 10550
+P 6775 10550
+F 0 "TP14" V 6950 10550 50  0000 L CNN
+F 1 "GND" V 7025 10550 50  0000 L CNN
+F 2 "TestPoint:TestPoint_Pad_D1.5mm" H 6975 10550 50  0001 C CNN
+F 3 "~" H 6975 10550 50  0001 C CNN
+F 4 "ok" H 6775 10550 50  0001 C CNN "Vorrätig"
+	1    6775 10550
 	0    1    1    0
 $EndComp
@@
 Wire Wire Line
 	7075 7125 7250 7125
-Wire Wire Line
-	6975 10550 7125 10550
-Connection ~ 6975 10550
-Wire Wire Line
-	6975 10100 7125 10100
-Connection ~ 6975 10100
 Connection ~ 2750 8650
 Wire Wire Line
@@
 Connection ~ 11700 4225
 Wire Wire Line
-	6575 10100 6975 10100
-Wire Wire Line
-	6575 10550 6975 10550
-Wire Wire Line
 	5775 6275 5775 6675
 Wire Wire Line
@@
 Text GLabel 9175 3075 0    50   Input ~ 0
 VDD_SD
-Wire Bus Line
-	8475 1225 8475 4825
 Text Label 5075 1375 0    50   ~ 0
 RST
@@
 Text Label 1425 3700 0    50   ~ 0
 VBUS
+Wire Wire Line
+	6575 10100 6775 10100
+Wire Wire Line
+	6575 10550 6775 10550
+Wire Wire Line
+	1325 2625 1325 3700
+$Comp
+L Connector:Conn_01x02_Male J5
+U 1 1 5FA7E015
+P 3225 3800
+F 0 "J5" H 3197 3682 50  0000 R CNN
+F 1 "CHG" H 3197 3773 50  0000 R CNN
+F 2 "Connector_PinHeader_2.54mm:PinHeader_1x02_P2.54mm_Vertical" H 3225 3800 50  0001 C CNN
+F 3 "~" H 3225 3800 50  0001 C CNN
+F 4 "ok" H 3225 3800 50  0001 C CNN "Vorrätig"
+	1    3225 3800
+	-1   0    0    1
+$EndComp
+Wire Wire Line
+	2575 3700 3025 3700
+Connection ~ 2575 3700
+$Comp
+L power:GND #PWR0112
+U 1 1 5FAE723C
+P 2975 3900
+F 0 "#PWR0112" H 2975 3650 50  0001 C CNN
+F 1 "GND" H 2975 3750 50  0000 C CNN
+F 2 "" H 2975 3900 50  0000 C CNN
+F 3 "" H 2975 3900 50  0000 C CNN
+	1    2975 3900
+	1    0    0    -1
+$EndComp
+Wire Wire Line
+	3025 3800 2975 3800
+Wire Wire Line
+	2975 3800 2975 3900
+$Comp
+L Diode:US1A D12
+U 1 1 5FC2072D
+P 12600 1300
+F 0 "D12" H 12600 1083 50  0000 C CNN
+F 1 "US1A" H 12600 1174 50  0000 C CNN
+F 2 "Diode_SMD:D_SMA" H 12600 1125 50  0001 C CNN
+F 3 "https://www.diodes.com/assets/Datasheets/ds16008.pdf" H 12600 1300 50  0001 C CNN
+	1    12600 1300
+	-1   0    0    1
+$EndComp
+Wire Wire Line
+	12450 1300 12425 1300
+Wire Bus Line
+	8475 1225 8475 4825
 $EndSCHEMATC
